File: hardware/kicad/fgl_g2/fgl_g2.kicad_pcb (KiCad board)
At the start: 2 copper layers, 90 x 60 mm, 73 parts, among them J1 USB-C (from bank), J10 XIAO socket 8-14, J2 POT 100k lin + SW, J3 LD2410S socket, J4 LD2410S cable, J5 PORT 1, J6 PORT 2, J7 PORT 3, J8 PORT 4, J9 XIAO socket 1-7, Q1 AO3400A, Q2 AO3401A, U2 TPS61500PWPR

Commit message: G2: fuse to 2 A hold (55 C derating), JLCPCB placement corrections, Flux second pass
F1: SMD1812B150TF/8 (1.06 A hold at 55 C) would trip at the 5 W cap in a
warm frame; now SMD1812B200TF/16 (C269145, ~1.58 A at 55 C), same 1812
footprint. make_cpl.py: every part at its pad-bbox centre (JLCPCB's origin;
KiCad's is pin 1 for headers, sockets, JST, ports, off-centre for the USB-C)
and rotations keyed by LCSC part, checked against JLCPCB's first preview:
J4/J5-J8 +180, JP1/JP2 +270, J1 0, SOT-23 180. Docs: supported strings up to
24 V total, USB-C 1.5 A source for full power, closed-frame G2-T2 run, new
G2-T14 radar through the glass, preview checklist; Flux's second pass saved
with resolutions.

Co-Authored-By: Claude Opus 5.5 <noreply@anthropic.com>
Claude-Session: https://claude.ai/code/session_013HVPKWJHmpHbXpMbmhYHhv
Parts:
- F1: value 1.5A hold -> 2A hold
Changed lines of the file:
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@@
 			)
 		)
-		(property "Value" "1.5A hold"
+		(property "Value" "2A hold"
 			(at 0 2.65 270)
 			(layer "F.Fab")
@@
 			)
 		)
-		(property "Datasheet" "https://datasheet.lcsc.com/datasheet/pdf/39c533899a45d694a011d998323027fc.pdf"
+		(property "Datasheet" "https://www.mouser.com/datasheet/2/447/2017100920153415341360-1516460.pdf"
 			(at 0 0 270)
 			(layer "F.Fab")
