File: hardware/kicad/fgl_g2/fgl_g2.kicad_sch (KiCad schematic)
At the start: 71 parts, among them J1 USB-C (from bank), J10 XIAO socket 8-14, J2 POT 100k lin + SW, J3 LD2410S socket, J4 LD2410S cable, J5 PORT 1, J6 PORT 2, J7 PORT 3, J8 PORT 4, J9 XIAO socket 1-7, Q1 AO3400A, Q2 AO3401A, U1 XIAO ESP32C3, U2 TPS61500PWPR

Commit message: G2: fix the Oct 24 audit findings; G2 firmware build with string guards
Hardware (schematic, PCB, fab outputs):
- R18 100k -> 2.2k so EN stays low through reset and USB flashing (H1)
- C5 10u 100V X7S 1210, C6 100n 100V (M2)
- R15 120k -> 110k: OVP 27.7 V, switch <= 35.1 V worst case (M3)
- JP1 solder jumper -> 1x3 2.54 mm header with a shunt (L1)
- Q2 soft start: R14 10k + new C16 100n gate-source (L2)
- Silkscreen: exact JP1 currents, pin-1 mark, "SWITCH OFF BEFORE WIRING PORTS"
- BOM tidy: U1 once, shunt line, voltages/tolerances in values;
  upload BOM in jlcpcb/ refreshed and kept in sync by build.sh

Firmware (src/main.c, platformio env seeed_xiao_esp32c3_g2):
- G2 pins, analog dimming, JP1 ceiling read, 5 W cap
- low-current start probe, open/short/window guards with NVS-learned
  window and relearn gesture, 30 s retry
- pot 1.85 V clamp, radar UART pull-ups, task watchdog (G1 M1/L2/L4)

Docs: g2_decisions.md D16 and updated values/tests, audit resolution,
hardware.md setup steps, README status, ERC summary.

Co-Authored-By: Claude Opus 5.5 <noreply@anthropic.com>
Claude-Session: https://claude.ai/code/session_013HVPKWJHmpHbXpMbmhYHhv
Parts:
- added C16: 100n 16V, Capacitor_SMD:C_0402_1005Metric, symbol Device:C_Small
- C11, C12, C14, C15, C3, C8, C9: value 100n -> 100n 50V
- C5: value 10u 50V -> 10u 100V; footprint Capacitor_SMD:C_1206_3216Metric -> Capacitor_SMD:C_1210_3225Metric; LCSC C89632 -> C576517; MPN CL31B106KBHNNNE -> GRM32EC72A106KE05L; Manufacturer Samsung -> Murata
- C6: value 100n -> 100n 100V; LCSC C14663 -> C15725; MPN CC0603KRX7R9BB104 -> CL10B104KC8NNNC; Manufacturer YAGEO -> Samsung
- C7: value 1u -> 1u 50V
- JP1: value 500mA -> ISEL; footprint Jumper:SolderJumper-3_P1.3mm_Open_RoundedPad1.0x1.5mm -> Connector_PinHeader_2.54mm:PinHeader_1x03_P2.54mm_Vertical; symbol Jumper:SolderJumper_3_Open -> Connector_Generic:Conn_01x03; LCSC (none) -> C49257; MPN solder jumper -> 2.54-1*3P; Manufacturer PCB -> BOOMELE
- R10: value 100R -> 100R 1%
- R11, R13, R23, R7: value 100k -> 100k 1%
- R12: value 33R 1W 2512 -> 33R 1% 1W
- R14: value 1k -> 10k 1%; LCSC C21190 -> C25804; MPN 0603WAF1001T5E -> 0603WAF1002T5E
- R15: value 120k 1% -> 110k 1%; LCSC C25808 -> C25805; MPN 0603WAF1203T5E -> 0603WAF1103T5E
- R17, R22, R26, R27, R28, R6: value 1k -> 1k 1%
- R18: value 100k -> 2.2k 1%; LCSC C25803 -> C4190; MPN 0603WAF1003T5E -> 0603WAF2201T5E
Connections:
- net Q2_G: now also C16.2
- net VBUS_F: now also C16.1
Other:
- note added: "D4 feeds the XIAO's 5V pin and blocks back-feed from its own USB-C. D6 (GPIO21) is UART0 TX: it toggles during boot, so ISEL goes through R22. D7 (GPIO20, UART0 RX) drives EN. GPIO20 has a ~45 k pull-up at reset, so R18 is 2.2 k: EN stays below 0.4 V until the firmware drives it (also in download mode). Strapping pins D0/D8/D9 unconnected. J9/J10: 5 mm low-profile sockets (JLCPCB fits them); the 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"
- note added: "Fill ports in order from PORT 1. Each filament: + wire -> its port's +, - wire -> NEXT, except the LAST filament's - wire -> END (PORT 4's NEXT is END too). Longest string 24 V. WIRE PORTS ONLY WITH THE POWER SWITCH OFF: an open string holds VOUT near OVP. Open or reversed filament: VOUT near OVP, firmware turns U2 off and retries at low current."
- note added: "I_max = 0.2 V / Rs. JP1 is a 2.54 mm header with one shunt: 2-3: R20 only, 244 mA; ISEL low. 1-2: R21 in parallel, 488 mA; ISEL high (R23). none: 244 mA; ISEL high, so the firmware assumes 488 and under-drives (safe)."
- note added: "Power switch: the pot's switch (J2 pin 4) pulls SW_N to GND. ON: Rd (R1/R2 5.1 k) reach GND, so a USB-C bank sees a sink attach and turns VBUS on; Q2's gate goes low and Q2 connects VBUS_F to +5V. OFF: Rd float (bank sees nothing attached, sleeps) and R13 holds Q2 off, which also cuts non-compliant banks and USB-A to C cables. Soft start: R14 10 k with C16 100 nF ramps Q2's gate over ~1 ms, so +5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"
- note added: "SEPIC: +5V -> L1 -> SW (switch) ; C4 couples SW to SEP_B ; L2 SEP_B -> GND ; D5 SEP_B -> VOUT. Works for any string from one 3 V filament (~2.7 V) to 24 V, and C4 blocks DC: no current path from the bank to the LEDs when U2 is off. f = 1.17 MHz (R19 82 k). OVP = 1.229 x (1 + 110k/5.1k) = 27.7 V (29.1 V worst case); switch sees VIN + VOUT + VD <= 35.1 V worst case (40 V abs max). L1 = L2 = 10 uH, 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"
- note added: "VSENSE = VOUT / 13: 27.7 V (OVP) -> 2.13 V, inside the C3's ADC range at 11 dB. Firmware uses it for: - P_LED = VOUT x I_set, capped at 5 W - open string or reversed filament (VOUT > 25.5 V, near OVP): EN off, retry - shorted output (VOUT ~ 0 while lit) - each start: 10 % current first, VOUT checked against the learned window - what is connected (one 12 V ~ 11 V, 3 x 3 V ~ 8.4 V) 0 uA when the dr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"
- note removed: "D4 feeds the XIAO's 5V pin and blocks back-feed from its own USB-C. D6 (GPIO21) is UART0 TX: it toggles during boot, so ISEL goes through R22. D7 (GPIO20, UART0 RX, input at boot) drives EN; R18 keeps it low until set. Strapping pins D0/D8/D9 unconnected. J9/J10: 5 mm low-profile sockets (JLCPCB fits them); the XIAO's USB-C faces the board edge."
- note removed: "Fill ports in order from PORT 1. Each filament: + wire -> its port's +, - wire -> NEXT, except the LAST filament, whose - wire goes to END. PORT 4's NEXT is also END. Mix 3 V and 12 V filaments freely; same current through all. Open string -> VOUT rises to OVP and firmware flags it (VSENSE). Silkscreen: + / NEXT / END on each port."
- note removed: "I_max = 0.2 V / Rs. JP1 open: R20 only, 244 mA. Bridge ALL THREE pads of JP1: R21 in parallel (488 mA) and ISEL to GND so the firmware knows."
- note removed: "Power switch: the pot's switch (J2 pin 4) pulls SW_N to GND. ON: Rd (R1/R2 5.1 k) reach GND, so a USB-C bank sees a sink attach and turns VBUS on; Q2's gate goes low and Q2 connects VBUS_F to +5V. OFF: Rd float (bank sees nothing attached, sleeps) and R13 holds Q2 off, which also cuts non-compliant banks and USB-A to C cables. The switch carries < 0.1 mA. R14 keeps cable ESD off Q2's gate. F1: 1.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"
- note removed: "SEPIC: +5V -> L1 -> SW (switch) ; C4 couples SW to SEP_B ; L2 SEP_B -> GND ; D5 SEP_B -> VOUT. Works for any string from one 3 V filament (~2.7 V) to ~28 V, and C4 blocks DC: no current path from the bank to the LEDs when U2 is off. f = 1.17 MHz (R19 82 k). OVP = 1.229 x (1 + 120k/5.1k) = 30.2 V; switch sees VIN + VOUT + VD < 36 V (40 V abs max). L1 = L2 = 10 uH, 4.1 A sat. Dimming: 19.5 kHz PWM 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"
- note removed: "VSENSE = VOUT / 13: 30.2 V (OVP) -> 2.32 V, inside the C3's ADC range at 11 dB. Firmware uses it for: - P_LED = VOUT x I_set, capped at 5 W - open string (VOUT near OVP at low current) - shorted output (VOUT ~ 0 while lit) - what is connected (one 12 V ~ 11 V, 3 x 3 V ~ 8.4 V) 0 uA when the driver is off (C4 blocks DC). R26-R28: 1 k series on the radar lines (ESD on the cable/socket)."

Commit message: G2: JP2 radar/manual mode jumper (D18)
- JP2 1x3 header (same part as JP1) on XIAO D8/GPIO8: shunt 1-2 = manual
  (radar ignored, lit whenever switched on, pot dims), 2-3 or none = radar.
- No external pull-up (no room by J10): the firmware enables GPIO8's
  internal pull-up and reads the jumper at power-on.
- Layout: JP2 at (114.54, 130), B.Cu route from J10 pin 2, silkscreen
  legend; C11 reference nudged. DRC 0/0, verify_pcb 184 pads.
- Netlist 42 nets / 175 connections / 73 parts; fab outputs, BOM (61
  placements, two loose shunts), assembly drawing, renders regenerated.
- Firmware: manual mode in the G2 build (start check, guards and 5 W cap
  unchanged; no off-delay or radar sleep). Compile-checked with -Werror.
- Docs: D18, pin tables, setup steps, bring-up test G2-T12.

Co-Authored-By: Claude Opus 5.5 <noreply@anthropic.com>
Claude-Session: https://claude.ai/code/session_013HVPKWJHmpHbXpMbmhYHhv
Parts:
- added JP2: RADAR_MODE, Connector_PinHeader_2.54mm:PinHeader_1x03_P2.54mm_Vertical, symbol Connector_Generic:Conn_01x03
Connections:
- net GND: now also JP2.1 (Pin_1)
- net RADAR_MODE: now reaches U1.9 (D8_GPIO8)
- net RADAR_MODE: now also J10.2 (Pin_2), JP2.2 (Pin_2)
- no-connect marks 12 -> 11
Other:
- note added: "D4 feeds the XIAO's 5V pin and blocks back-feed from its own USB-C. D6 (GPIO21) is UART0 TX: it toggles during boot, so ISEL goes through R22. D7 (GPIO20, UART0 RX) drives EN. GPIO20 has a ~45 k pull-up at reset, so R18 is 2.2 k: EN stays below 0.4 V until the firmware drives it (also in download mode). D8 (GPIO8) reads JP2 with its internal pull-up: low = manual mode (radar ignored). Strapping p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"
- note removed: "D4 feeds the XIAO's 5V pin and blocks back-feed from its own USB-C. D6 (GPIO21) is UART0 TX: it toggles during boot, so ISEL goes through R22. D7 (GPIO20, UART0 RX) drives EN. GPIO20 has a ~45 k pull-up at reset, so R18 is 2.2 k: EN stays below 0.4 V until the firmware drives it (also in download mode). Strapping pins D0/D8/D9 unconnected. J9/J10: 5 mm low-profile sockets (JLCPCB fits them); the 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"
Changed lines of the file:
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@@
 	(title_block
 		(title "Fused Glass Lighting controller")
-		(date "2026-10-24")
+		(date "2026-10-27")
 		(rev "G2")
 		(company "Rob Lim")
@@
 		)
 	)
-	(text "D4 feeds the XIAO's 5V pin and blocks back-feed from its own USB-C.\nD6 (GPIO21) is UART0 TX: it toggles during boot, so ISEL goes through R22.\nD7 (GPIO20, UART0 RX) drives EN. GPIO20 has a ~45 k pull-up at reset, so R18 is\n2.2 k: EN stays below 0.4 V until the firmware drives it (also in download mode).\nStrapping pins D0/D8/D9 unconnected. J9/J10: 5 mm low-profile sockets\n(JLCPCB fits them); the XIAO's USB-C faces the board edge."
+	(text "D4 feeds the XIAO's 5V pin and blocks back-feed from its own USB-C.\nD6 (GPIO21) is UART0 TX: it toggles during boot, so ISEL goes through R22.\nD7 (GPIO20, UART0 RX) drives EN. GPIO20 has a ~45 k pull-up at reset, so R18 is\n2.2 k: EN stays below 0.4 V until the firmware drives it (also in download mode).\nD8 (GPIO8) reads JP2 with its internal pull-up: low = manual mode\n(radar ignored). Strapping pin, but only in download mode: move the\nshunt off 1-2 before forcing download with BOOT. D0/D9 unconnected. J9/J10: 5 mm low-profile sockets\n(JLCPCB fits them); the XIAO's USB-C faces the board edge."
 		(exclude_from_sim no)
 		(at 50.8 182.88 0)
@@
 		)
 	)
-	(text "Power: 5 V from the bank via Q2. LED power capped at 5 W in firmware\n(~1.4 A from the bank); 1.7 W lit at prototype brightness; idle ~4 mA\nwith keep-alive, ~0.7 mA without (model: power_model.py).\n\nPins (XIAO):\n  D1 GPIO3  ADC_POT    ADC1_CH3\n  D2 GPIO4  VSENSE     ADC1_CH4, VOUT / 13\n  D3 GPIO5  RADAR_OT2  wake, high = present\n  D4 GPIO6  UART_TX -> radar RX (115200 8N1)\n  D5 GPIO7  UART_RX <- radar OT1/TX\n  D6 GPIO21 ISEL_IO    low = 244 mA (shunt 2-3), via R22\n  D7 GPIO20 DIM_PWM    LEDC 19.5 kHz -> EN (analog dim)\n  D10 GPIO10 KA_DRV    keep-alive gate\n\nAssembly: JLCPCB fits everything incl. through-hole J2-J8 and the\nXIAO sockets; you plug in the XIAO and the radar. DNP: D1.\n\nBring-up (docs/g2_decisions.md): SEPIC at the extremes (one 3 V\nfilament at 244 mA; 24 V string at the 5 W cap), filament\ntemperature in the frame, bank wake via the switch."
+	(text "Power: 5 V from the bank via Q2. LED power capped at 5 W in firmware\n(~1.4 A from the bank); 1.7 W lit at prototype brightness; idle ~4 mA\nwith keep-alive, ~0.7 mA without (model: power_model.py).\n\nPins (XIAO):\n  D1 GPIO3  ADC_POT    ADC1_CH3\n  D2 GPIO4  VSENSE     ADC1_CH4, VOUT / 13\n  D3 GPIO5  RADAR_OT2  wake, high = present\n  D4 GPIO6  UART_TX -> radar RX (115200 8N1)\n  D5 GPIO7  UART_RX <- radar OT1/TX\n  D6 GPIO21 ISEL_IO    low = 244 mA (shunt 2-3), via R22\n  D7 GPIO20 DIM_PWM    LEDC 19.5 kHz -> EN (analog dim)\n  D8 GPIO8  RADAR_MODE   JP2 1-2 = manual, 2-3/none = radar\n  D10 GPIO10 KA_DRV    keep-alive gate\n\nAssembly: JLCPCB fits everything incl. through-hole J2-J8 and the\nXIAO sockets; you plug in the XIAO and the radar. DNP: D1.\n\nBring-up (docs/g2_decisions.md): SEPIC at the extremes (one 3 V\nfilament at 244 mA; 24 V string at the 5 W cap), filament\ntemperature in the frame, bank wake via the switch."
 		(exclude_from_sim no)
 		(at 309.88 29.21 0)
@@
 	)
 	(no_connect
-		(at 121.92 172.72)
-	)
-	(no_connect
-		(at 86.36 154.94)
-	)
-	(no_connect
 		(at 48.26 76.2)
 	)
@@
 	)
 	(wire
+		(pts
+			(xy 86.36 154.94) (xy 88.9 154.94)
+		)
+		(stroke
+			(width 0)
+			(type default)
+		)
+	)
+	(label "RADAR_MODE"
+		(at 88.9 154.94 0)
+		(effects
+			(font
+				(size 1.27 1.27)
+			)
+			(justify left bottom)
+		)
+	)
+	(wire
+		(pts
+			(xy 121.92 172.72) (xy 121.92 175.26)
+		)
+		(stroke
+			(width 0)
+			(type default)
+		)
+	)
+	(label "RADAR_MODE"
+		(at 121.92 175.26 270)
+		(effects
+			(font
+				(size 1.27 1.27)
+			)
+			(justify right bottom)
+		)
+	)
+	(symbol
+		(lib_id "Connector_Generic:Conn_01x03")
+		(at 104.14 177.8 0)
+		(unit 1)
+		(exclude_from_sim no)
+		(in_bom yes)
+		(on_board yes)
+		(dnp no)
+		(property "Reference" "JP2"
+			(at 104.14 172.72 0)
+			(effects
+				(font
+					(size 1.27 1.27)
+				)
+				(justify left)
+			)
+		)
+		(property "Value" "RADAR_MODE"
+			(at 104.14 182.88 0)
+			(effects
+				(font
+					(size 1.27 1.27)
+				)
+				(justify left)
+			)
+		)
+		(property "Footprint" "Connector_PinHeader_2.54mm:PinHeader_1x03_P2.54mm_Vertical"
+			(at 104.14 177.8 0)
+			(effects
+				(font
+					(size 1.27 1.27)
+				)
+				(hide yes)
+			)
+		)
+		(property "Datasheet" ""
+			(at 104.14 177.8 0)
+			(effects
+				(font
+					(size 1.27 1.27)
+				)
+				(hide yes)
+			)
+		)
+		(property "Description" "2.54 mm 1x3 pin header with a shunt: 1-2 manual (no radar), 2-3 radar"
+			(at 104.14 177.8 0)
+			(effects
+				(font
+					(size 1.27 1.27)
+				)
+			)
+		)
+		(property "LCSC" "C49257"
+			(at 104.14 177.8 0)
+			(effects
+				(font
+					(size 1.27 1.27)
+				)
+				(hide yes)
+			)
+		)
+		(property "MPN" "2.54-1*3P"
+			(at 104.14 177.8 0)
+			(effects
+				(font
+					(size 1.27 1.27)
+				)
+				(hide yes)
+			)
+		)
+		(property "Manufacturer" "BOOMELE"
+			(at 104.14 177.8 0)
+			(effects
+				(font
+					(size 1.27 1.27)
+				)
+				(hide yes)
+			)
+		)
+		(pin "1"
+		)
+		(pin "2"
+		)
+		(pin "3"
+		)
+		(instances
+			(project "fgl_g2"
+				(path "/ab8fe160-4d5e-53d4-be1b-69cfad966fcd"
+					(reference "JP2")
+					(unit 1)
+				)
+			)
+		)
+	)
+	(wire
+		(pts
+			(xy 99.06 175.26) (xy 96.52 175.26)
+		)
+		(stroke
+			(width 0)
+			(type default)
+		)
+	)
+	(symbol
+		(lib_id "power:GND")
+		(at 96.52 175.26 270)
+		(unit 1)
+		(exclude_from_sim no)
+		(in_bom yes)
+		(on_board yes)
+		(dnp no)
+		(property "Reference" "#PWR059"
+			(at 90.17 175.26 0)
+			(effects
+				(font
+					(size 1.27 1.27)
+				)
+				(hide yes)
+			)
+		)
+		(property "Value" "GND"
+			(at 92.71 175.26 0)
+			(effects
+				(font
+					(size 1.27 1.27)
+				)
+				(hide yes)
+			)
+		)
+		(property "Footprint" ""
+			(at 104.14 181.61 0)
+			(effects
+				(font
+					(size 1.27 1.27)
+				)
+				(hide yes)
+			)
+		)
+		(property "Datasheet" ""
+			(at 104.14 181.61 0)
+			(effects
+				(font
+					(size 1.27 1.27)
+				)
+				(hide yes)
+			)
+		)
+		(property "Description" ""
+			(at 104.14 181.61 0)
+			(effects
+				(font
+					(size 1.27 1.27)
+				)
+			)
+		)
+		(pin "1"
+		)
+		(instances
+			(project "fgl_g2"
+				(path "/ab8fe160-4d5e-53d4-be1b-69cfad966fcd"
+					(reference "#PWR059")
+					(unit 1)
+				)
+			)
+		)
+	)
+	(wire
+		(pts
+			(xy 99.06 177.8) (xy 88.9 177.8)
+		)
+		(stroke
+			(width 0)
+			(type default)
+		)
+	)
+	(label "RADAR_MODE"
+		(at 88.9 177.8 180)
+		(effects
+			(font
+				(size 1.27 1.27)
+			)
+			(justify right bottom)
+		)
+	)
+	(no_connect
+		(at 99.06 180.34)
+	)
+	(wire
