File: hardware/kicad/fgl_g2/fgl_g2.kicad_sch (KiCad schematic)
At the start: 74 parts, among them J1 USB-C (from bank), J10 XIAO socket 8-14, J2 POT 100k lin + SW, J3 LD2410S socket, J4 LD2410S cable, J5 PORT 1, J6 PORT 2, J7 PORT 3, J8 PORT 4, J9 XIAO socket 1-7, Q1 AO3400A, Q2 AO3401A, U1 XIAO ESP32C3, U2 TPS61500PWPR

Commit message: G2: C4 to its basic X5R equivalent, ports ordered as DEGSON DG212R (JL212R short)
C4: CL31A106KBHNNNE (C13585, JLCPCB basic) for CL31B106KBHNNNE; saves an
extended-part fee. J5-J8: DEGSON DG212R-THR-3.5-03P (C7603454), the same-size
alternative from D19, because JLCPCB is 12 JL212R short; its JLCPCB rotation
is marked unverified in make_cpl.py. No other extended part has a basic
equivalent even with a layout change (reasons in D19's cost follow-up).

Co-Authored-By: Claude Opus 5.5 <noreply@anthropic.com>
Claude-Session: https://claude.ai/code/session_013HVPKWJHmpHbXpMbmhYHhv
Parts:
- C4: LCSC C89632 -> C13585; MPN CL31B106KBHNNNE -> CL31A106KBHNNNE
- J5, J6, J7, J8: LCSC C2962951 -> C7603454; MPN JL212R-35003B01 -> DG212R-THR-3.5-03P-13-1000A(H); Manufacturer JILN -> DEGSON
Changed lines of the file:
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@@
 			)
 		)
-		(property "Datasheet" "https://datasheet.lcsc.com/datasheet/pdf/edf099acf8994a482e4343677e6896d8.pdf"
+		(property "Datasheet" "https://atta.szlcsc.com/upload/public/pdf/source/20230907/20A31750C0F42741679442E51C870286.pdf?Expires=4070880000&OSSAccessKeyId=LTAIJDIkh7KmGS1H&Signature=bC5y63SvwdXcuwa1uZSa1Htf5PQ%3D&response-content-disposition=attachment%3Bfilename%3DC7603454_%25E5%25BC%25B9%25E7%25B0%25A7%25E5%25BC%258F%25E6%258E%25A5%25E7%25BA%25BF%25E7%25AB%25AF%25E5%25AD%2590_DG212R-THR-3.5-03P-13-1000A%2528H%2529_%25E8%25A7%2584%25E6%25A0%25BC%25E4%25B9%25A6_WJ458111.PDF"
 			(at 215.9 157.48 0)
 			(effects
@@
 			)
 		)
-		(property "LCSC" "C2962951"
+		(property "LCSC" "C7603454"
 			(at 215.9 157.48 0)
 			(effects
@@
 			)
 		)
-		(property "MPN" "JL212R-35003B01"
+		(property "MPN" "DG212R-THR-3.5-03P-13-1000A(H)"
 			(at 215.9 157.48 0)
 			(effects
@@
 			)
 		)
-		(property "Manufacturer" "JILN"
+		(property "Manufacturer" "DEGSON"
 			(at 215.9 157.48 0)
 			(effects
@@
 			)
 		)
-		(property "Datasheet" "https://datasheet.lcsc.com/datasheet/pdf/edf099acf8994a482e4343677e6896d8.pdf"
+		(property "Datasheet" "https://atta.szlcsc.com/upload/public/pdf/source/20230907/20A31750C0F42741679442E51C870286.pdf?Expires=4070880000&OSSAccessKeyId=LTAIJDIkh7KmGS1H&Signature=bC5y63SvwdXcuwa1uZSa1Htf5PQ%3D&response-content-disposition=attachment%3Bfilename%3DC7603454_%25E5%25BC%25B9%25E7%25B0%25A7%25E5%25BC%258F%25E6%258E%25A5%25E7%25BA%25BF%25E7%25AB%25AF%25E5%25AD%2590_DG212R-THR-3.5-03P-13-1000A%2528H%2529_%25E8%25A7%2584%25E6%25A0%25BC%25E4%25B9%25A6_WJ458111.PDF"
 			(at 276.86 157.48 0)
 			(effects
@@
 			)
 		)
-		(property "LCSC" "C2962951"
+		(property "LCSC" "C7603454"
 			(at 276.86 157.48 0)
 			(effects
@@
 			)
 		)
-		(property "MPN" "JL212R-35003B01"
+		(property "MPN" "DG212R-THR-3.5-03P-13-1000A(H)"
 			(at 276.86 157.48 0)
 			(effects
@@
 			)
 		)
-		(property "Manufacturer" "JILN"
+		(property "Manufacturer" "DEGSON"
 			(at 276.86 157.48 0)
 			(effects
@@
 			)
 		)
-		(property "Datasheet" "https://datasheet.lcsc.com/datasheet/pdf/edf099acf8994a482e4343677e6896d8.pdf"
+		(property "Datasheet" "https://atta.szlcsc.com/upload/public/pdf/source/20230907/20A31750C0F42741679442E51C870286.pdf?Expires=4070880000&OSSAccessKeyId=LTAIJDIkh7KmGS1H&Signature=bC5y63SvwdXcuwa1uZSa1Htf5PQ%3D&response-content-disposition=attachment%3Bfilename%3DC7603454_%25E5%25BC%25B9%25E7%25B0%25A7%25E5%25BC%258F%25E6%258E%25A5%25E7%25BA%25BF%25E7%25AB%25AF%25E5%25AD%2590_DG212R-THR-3.5-03P-13-1000A%2528H%2529_%25E8%25A7%2584%25E6%25A0%25BC%25E4%25B9%25A6_WJ458111.PDF"
 			(at 185.42 157.48 0)
 			(effects
@@
 			)
 		)
-		(property "LCSC" "C2962951"
+		(property "LCSC" "C7603454"
 			(at 185.42 157.48 0)
 			(effects
@@
 			)
 		)
-		(property "MPN" "JL212R-35003B01"
+		(property "MPN" "DG212R-THR-3.5-03P-13-1000A(H)"
 			(at 185.42 157.48 0)
 			(effects
@@
 			)
 		)
-		(property "Manufacturer" "JILN"
+		(property "Manufacturer" "DEGSON"
 			(at 185.42 157.48 0)
 			(effects
@@
 			)
 		)
-		(property "Datasheet" "https://datasheet.lcsc.com/datasheet/pdf/a1390a51092e4f3c84866ab492516a00.pdf"
+		(property "Datasheet" "https://datasheet.lcsc.com/datasheet/pdf/02336ea48ea44ca18c72517dd3cb7b47.pdf"
 			(at 255.27 45.72 0)
 			(effects
@@
 			)
 		)
-		(property "LCSC" "C89632"
+		(property "LCSC" "C13585"
 			(at 255.27 45.72 0)
 			(effects
@@
 			)
 		)
-		(property "MPN" "CL31B106KBHNNNE"
+		(property "MPN" "CL31A106KBHNNNE"
 			(at 255.27 45.72 0)
 			(effects
@@
 			)
 		)
-		(property "Datasheet" "https://datasheet.lcsc.com/datasheet/pdf/edf099acf8994a482e4343677e6896d8.pdf"
+		(property "Datasheet" "https://atta.szlcsc.com/upload/public/pdf/source/20230907/20A31750C0F42741679442E51C870286.pdf?Expires=4070880000&OSSAccessKeyId=LTAIJDIkh7KmGS1H&Signature=bC5y63SvwdXcuwa1uZSa1Htf5PQ%3D&response-content-disposition=attachment%3Bfilename%3DC7603454_%25E5%25BC%25B9%25E7%25B0%25A7%25E5%25BC%258F%25E6%258E%25A5%25E7%25BA%25BF%25E7%25AB%25AF%25E5%25AD%2590_DG212R-THR-3.5-03P-13-1000A%2528H%2529_%25E8%25A7%2584%25E6%25A0%25BC%25E4%25B9%25A6_WJ458111.PDF"
 			(at 246.38 157.48 0)
 			(effects
@@
 			)
 		)
-		(property "LCSC" "C2962951"
+		(property "LCSC" "C7603454"
 			(at 246.38 157.48 0)
 			(effects
@@
 			)
 		)
-		(property "MPN" "JL212R-35003B01"
+		(property "MPN" "DG212R-THR-3.5-03P-13-1000A(H)"
 			(at 246.38 157.48 0)
 			(effects
@@
 			)
 		)
-		(property "Manufacturer" "JILN"
+		(property "Manufacturer" "DEGSON"
 			(at 246.38 157.48 0)
 			(effects

Commit message: docs: G2 off-board parts sourcing; U1 MPN is the pre-soldered XIAO
- New docs/g2_sourcing.md: where to buy the pot, knob, filaments, XIAO,
  LD2410S, USB-C panel extension and power bank for 5-10 frames, the
  recessed pot geometry for the 20 mm frame wall, and bank safety notes
- Pot: Same Sky PTN09S1-H100115K1B (knurled shaft) with a push-on Cliff
  K21 knob, so the knob can sit in a recess with no set screw to reach
- U1 MPN 113991054 (no headers) -> 102010633 (pre-soldered) in the
  schematic, netlist, BOM, gen_g2.py and g2_expected.py; PDF re-exported
- New bring-up test G2-T15: the chosen bank in the closed frame

Co-Authored-By: Claude Opus 5.5 <noreply@anthropic.com>
Claude-Session: https://claude.ai/code/session_013HVPKWJHmpHbXpMbmhYHhv
Parts:
- U1: MPN 113991054 -> 102010633
Changed lines of the file:
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@@
 			)
 		)
-		(property "MPN" "113991054"
+		(property "MPN" "102010633"
 			(at 63.5 160.02 0)
 			(effects
